File: PCB/Energy Monitor/CTClamps.kicad_sch (KiCad schematic)
At the start: 54 parts

Commit message: slow progress
Parts:
- C? (x8): footprint (none) -> Capacitor_SMD:C_0603_1608Metric_Pad1.08x0.95mm_HandSolder
- C? (x2): value (none) -> 100n; footprint (none) -> Capacitor_SMD:C_0603_1608Metric_Pad1.08x0.95mm_HandSolder
- C?: value (none) -> C; footprint (none) -> Capacitor_SMD:C_0603_1608Metric_Pad1.08x0.95mm_HandSolder
- R? (x16): footprint (none) -> Resistor_SMD:R_0603_1608Metric_Pad0.98x0.95mm_HandSolder
- R? (x4): footprint (none) -> Resistor_SMD:R_1210_3225Metric_Pad1.30x2.65mm_HandSolder
- R? (x4): footprint (none) -> Resistor_THT:R_Axial_DIN0207_L6.3mm_D2.5mm_P10.16mm_Horizontal
- U? (x6): value (none) -> TL072
