File: PCB/Energy Monitor/PulseMeter.kicad_sch (KiCad schematic)
At the start: 0 parts

Commit message: slow progress
Parts:
- added C?: C, Capacitor_SMD:C_1206_3216Metric_Pad1.33x1.80mm_HandSolder, symbol Device:C
- added D?: LED, LED_SMD:LED_0603_1608Metric_Pad1.05x0.95mm_HandSolder, symbol Device:LED
- added D?: D_Photo, symbol Device:D_Photo
- added H? (x3): MountingHole_Pad, symbol Mechanical:MountingHole_Pad
- added Q?: BC807, Package_TO_SOT_SMD:SOT-23, symbol Transistor_BJT:BC807
- added Q?: 2SC4213, Package_TO_SOT_SMD:SOT-323_SC-70, symbol Transistor_BJT:2SC4213
- added R? (x6): R, Resistor_SMD:R_0603_1608Metric_Pad0.98x0.95mm_HandSolder, symbol Device:R
- added R?: 1K, Resistor_SMD:R_0603_1608Metric_Pad0.98x0.95mm_HandSolder, symbol Device:R
Connections:
- new net: Q?.1 (B), R?.2
- new net: Q?.2 (E), R?.1, R?.2
- new net: Q?.3 (C), R?.1, R?.1
- new net: C?.2, H?.1, Q?.2 (E), R?.2, R?.2
- new net: D?.2 (A), Q?.1 (B), R?.1
- new net: D?.1 (K), Q?.3 (C), R?.1
- new net: D?.2 (A), R?.2
- new net: C?.1, D?.1 (K), H?.1, R?.1, R?.1
- new net PULSE: H?.1, R?.2, R?.2
Other:
- note added: "GND"
- note added: "PULSE"
- note added: "Pulse Meter"
- note added: "Pulse meter for meters which have a pulsing LED as the output. Saves a CT clamp or allows live calibration of the values by comparing the Pulse and CT clamp readings. Optical Pluse meter sensor on seperate part of PCB which can be seperated and broken off. Connected here to allow it to be on one PCB and for cheap China fab houses to not see it as a panel and charge more money for fabrication. Sou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"
- note added: "VCC"
