File: PCB/Energy Monitor/ac.kicad_sch (KiCad schematic)
At the start: 34 parts

Commit message: slow progress
Parts:
- added C?: C, Capacitor_SMD:C_0603_1608Metric_Pad1.08x0.95mm_HandSolder, symbol Device:C
- added D?: ~, symbol Device:D_Zener
- added D?: LED, LED_SMD:LED_0603_1608Metric_Pad1.05x0.95mm_HandSolder, symbol Device:LED
- added R? (x2): 470k, Resistor_SMD:R_0603_1608Metric_Pad0.98x0.95mm_HandSolder, symbol Device:R
- added R?: 1K, Resistor_SMD:R_0603_1608Metric_Pad0.98x0.95mm_HandSolder, symbol Device:R
- added R? (x2): 1k, Resistor_SMD:R_0603_1608Metric_Pad0.98x0.95mm_HandSolder, symbol Device:R
- J?: footprint (none) -> Connector_BarrelJack:BarrelJack_SwitchcraftConxall_RAPC10U_Horizontal
- J?: footprint (none) -> Connector_BarrelJack:BarrelJack_Wuerth_6941xx301002
Connections:
- net +3V3: now also R?.1, R?.1
- net GND: now also C?.2, D?.1 (K), D?.2 (A), R?.2
- net at U?.5 (+): now also R?.2
- net at U?.6 (-): now also C?.1, R?.1, R?.2
- net at U?.7: now also R?.1
- net AC_LV_L-Biased: now reaches R?.1, R?.1, R?.2
- net AC_LV_L-Biased: now also R?.1
- new net: D?.2 (A), R?.2
- new net Fmeas_AC: D?.1 (K), R?.2
Other:
- note added: "AC Frequency Measurement"
- note added: "Comparitor circuit to measure the AC frequency. This allows the use of a simple PWM or clock input on the microcontrolled with no extra zero crossing math logic nessesary."
- moved on the sheet: R?, U?B
