File: PCB/Energy Monitor/uController.kicad_sch (KiCad schematic)
At the start: 0 parts

Commit message: slow progress
Parts:
- added C?: 10u, Capacitor_SMD:C_0603_1608Metric_Pad1.08x0.95mm_HandSolder, symbol Device:C
- added C? (x3): 100n, Capacitor_SMD:C_0603_1608Metric_Pad1.08x0.95mm_HandSolder, symbol Device:C
- added C?: 1u, Capacitor_SMD:C_0603_1608Metric_Pad1.08x0.95mm_HandSolder, symbol Device:C
- added D? (x4): LED, LED_SMD:LED_0603_1608Metric_Pad1.05x0.95mm_HandSolder, symbol Device:LED
- added J?: Conn_01x04_Female, Connector_PinHeader_2.54mm:PinHeader_1x04_P2.54mm_Vertical, symbol Connector:Conn_01x04_Female
- added R? (x4): 1K, Resistor_SMD:R_0603_1608Metric_Pad0.98x0.95mm_HandSolder, symbol Device:R
- added R?: 10K, Resistor_SMD:R_0603_1608Metric_Pad0.98x0.95mm_HandSolder, symbol Device:R
- added SW? (x2): SW_Push, symbol Switch:SW_Push
- added U?: ESP32-S2-WROVER, RF_Module:ESP32-S2-WROVER, symbol RF_Module:ESP32-S2-WROVER
Connections:
- new net: D?.1 (K), U?.35 (IO41)
- new net: D?.2 (A), R?.2 (x4)
- new net: D?.1 (K), U?.33 (IO39)
- new net: D?.1 (K), U?.34 (IO40)
- new net: D?.1 (K), U?.36 (IO42)
- new net +3V3: C?.1, C?.1, J?.4 (Pin_4), R?.1, R?.1, R?.1, R?.1, R?.1, U?.2 (3V3)
- new net CHIP_PU: C?.1, C?.2, R?.2, SW?.2, U?.41 (EN)
- new net GND: C?.1, C?.1, C?.2, C?.2, C?.2, J?.1 (Pin_1), SW?.1, SW?.1, U?.1 (GND), U?.26 (GND), U?.42 (GND), U?.43 (GND)
- new net GPIO0: C?.2, SW?.2, U?.3 (IO00)
- new net GPIO17 / ADC2_6 / U1TXD: U?.20 (IO17)
- new net GPIO18 / ADC2-7 / U1RXD / DAC_2: U?.21 (IO18)
- new net RXD0: J?.3 (Pin_3), U?.38 (RXD0)
- new net TXD0: J?.2 (Pin_2), U?.37 (TXD0)
Other:
- note added: "I DONT TRUST THIS SYMBOL"
- note added: "https://dl.espressif.com/dl/schematics/ESP32-S2-DevKitM-1_V1_Schematics.pdf"
- note added: "https://docs.espressif.com/projects/esp-idf/en/latest/esp32s2/hw-reference/esp32s2/user-guide-devkitm-1-v1.html"
- note removed: "https://esp32.com/viewtopic.php?f=5&t=21992"
